Commit message: fix simulation

File: description/urdf/robot/robot_description.urdf.xacro (robot description, xacro)
@@ -6,4 +6,5 @@
     <xacro:property name="base_length" value="0.195"/>
     <xacro:property name="base_height" value="0.002"/>
+    <xacro:property name="base_mass" value="4.0" /> <!-- arbitrary value for base mass -->
     <xacro:property name="wheel_radius" value="0.0325"/>
     <xacro:property name="wheel_width" value="0.025"/>
@@ -13,7 +14,15 @@
     <xacro:property name="wheel_front_xoff" value="0.065"/>
     <xacro:property name="wheelbase" value="0.145"/>
+    <xacro:property name="wheel_mass" value="0.34055" /> <!-- arbitrary value for wheel mass -->
     <!-- Robot Base -->
     <link name="base_link">
+        <collision>
+            <origin xyz="0 0 0" rpy="0 0 0"/>
+            <geometry>
+                <box size="${base_length} ${base_width} ${base_height}"/>
+            </geometry>
+        </collision>
         <visual>
+            <origin xyz="0 0 0" rpy="0 0 0"/>
             <geometry>
                 <box size="${base_length} ${base_width} ${base_height}"/>
@@ -23,10 +32,18 @@
             </material>
         </visual>
+        <inertial>
+            <origin xyz="0 0 0" rpy="0 0 0"/>
+            <mass value="${base_mass}"/>
+                <inertia
+                ixx="0.000270" ixy="0.0" ixz="0.0"
+                iyy="0.000270" iyz="0.0"
+                izz="0.000426"/>
+        </inertial>
     </link>
     <!-- Robot Footprint -->
     <link name="base_footprint"/>
     <joint name="base_joint" type="fixed">
-        <parent link="base_link"/>
-        <child link="base_footprint"/>
+        <parent link="base_footprint"/>
+        <child link="base_link"/>
         <origin xyz="0.0 0.0 ${-(wheel_radius+wheel_zoff)}" rpy="0 0 0"/>
     </joint>
@@ -70,4 +87,10 @@
     <xacro:macro name="wheel" params="prefix x_reflect y_reflect">
         <link name="${prefix}_link">
+            <collision>
+                <origin xyz="0 0 0" rpy="${pi/2} 0 0"/>
+                <geometry>
+                    <cylinder length="${wheel_width}" radius="${wheel_radius}"/>
+                </geometry>
+            </collision>
             <visual>
             <origin xyz="0 0 0" rpy="${pi/2} 0 0"/>
@@ -79,4 +102,12 @@
             </material>
             </visual>
+            <inertial>
+                <origin xyz="0 0 0" rpy="${pi/2} 0 0"/>
+                <mass value="${wheel_mass}"/>
+                <inertia
+                    ixx="0.000270" ixy="0.0" ixz="0.0"
+                    iyy="0.000270" iyz="0.0"
+                    izz="0.000426"/>
+            </inertial>
         </link>
         <joint name="${prefix}_joint" type="continuous">
