Commit message: added description and bringup

File: description/urdf/robot.urdf.xacro (robot description, xacro)
@@ -6,11 +6,10 @@
   <xacro:arg name="prefix" default="" />
   <xacro:include filename="robot/robot_description.urdf.xacro" />
-  <!-- Import carlikebot ros2_control description
-  <xacro:include filename="$(find description)/ros2_control/robot.ros2_control.xacro" /> -->
+  <!-- Import carlikebot ros2_control description -->
+  <xacro:include filename="robot/robot.ros2_control.xacro" />
   <xacro:carlikebot />
-  <!-- <xacro:carlikebot_ros2_control
+  <xacro:carlikebot_ros2_control
     name="CarlikeBot"
-    prefix="$(arg prefix)"
     use_mock_hardware="$(arg use_mock_hardware)"
-    mock_sensor_commands="$(arg mock_sensor_commands)" /> -->
+    mock_sensor_commands="$(arg mock_sensor_commands)" />
 </robot>

File: description/urdf/robot/robot.ros2_control.xacro (robot description, xacro)
@@ -1,16 +1,15 @@
 <?xml version="1.0"?>
 <robot xmlns:xacro="http://www.ros.org/wiki/xacro">
-  <xacro:macro name="carlikebot_ros2_control" params="name prefix">
+  <xacro:macro name="carlikebot_ros2_control" params="name use_mock_hardware:=^|false mock_sensor_commands:=^|false">
     <ros2_control name="${name}" type="system">
       <hardware>
-        <plugin>my_bot/CarlikeBotSystemHardware</plugin>
-        <param name="example_param_hw_start_duration_sec">0</param>
-        <param name="example_param_hw_stop_duration_sec">3.0</param>
+        <plugin>mock_components/GenericSystem</plugin>
+        <param name="mock_sensor_commands">${mock_sensor_commands}</param>
       </hardware>
-      <joint name="${prefix}virtual_front_wheel_joint">
+      <joint name="virtual_front_wheel_joint">
         <command_interface name="position"/>
         <state_interface name="position"/>
       </joint>
-      <joint name="${prefix}virtual_rear_wheel_joint">
+      <joint name="virtual_rear_wheel_joint">
         <command_interface name="velocity"/>
         <state_interface name="velocity"/>

File: description/urdf/robot/robot_description.urdf.xacro (robot description, xacro)
@@ -53,10 +53,11 @@
             <parent link="base_link"/>
             <child link="virtual_${prefix}_wheel"/>
-            <origin xyz="${x_reflect*wheelbase/2} 0 -${base_height/2}" rpy="0 0 0"/>
             <xacro:if value="${x_reflect == -1}">
+                <origin xyz="${x_reflect*wheel_back_xoff} 0 ${-wheel_zoff}" rpy="0 0 0"/>
                 <axis xyz="1 0 0"/>
                 <limit effort="100.0" velocity="100.0"/>
             </xacro:if>
             <xacro:if value="${x_reflect == 1}">
+                <origin xyz="${wheel_front_xoff} 0 ${-wheel_zoff}" rpy="0 0 0"/>
                 <axis xyz="0 0 1"/>
                 <limit lower="-0.4" upper="0.4" effort="100.0" velocity="0.0"/>

Commit message: add imu sensor

File: description/urdf/robot.urdf.xacro (robot description, xacro)
@@ -4,5 +4,5 @@
   <xacro:arg name="use_mock_hardware" default="false" />
   <xacro:arg name="mock_sensor_commands" default="false" />
-  <xacro:arg name="prefix" default="" />
+  <!-- <xacro:arg name="prefix" default="" /> -->
   <xacro:include filename="robot/robot_description.urdf.xacro" />
   <!-- Import carlikebot ros2_control description -->

File: description/urdf/robot/robot.ros2_control.xacro (robot description, xacro)
@@ -1,9 +1,14 @@
 <?xml version="1.0"?>
 <robot xmlns:xacro="http://www.ros.org/wiki/xacro">
-  <xacro:macro name="carlikebot_ros2_control" params="name use_mock_hardware:=^|false mock_sensor_commands:=^|false">
+  <xacro:macro name="carlikebot_ros2_control" params="name use_mock_hardware:=^|false mock_sensor_commands:=^|false use_gazebo_classic:=^|false">
     <ros2_control name="${name}" type="system">
       <hardware>
-        <plugin>mock_components/GenericSystem</plugin>
-        <param name="mock_sensor_commands">${mock_sensor_commands}</param>
+        <xacro:if value="${use_gazebo_classic}">
+          <plugin>gazebo_ros2_control/GazeboSystem</plugin>
+        </xacro:if>
+        <xacro:if value="${use_mock_hardware}">
+          <plugin>mock_components/GenericSystem</plugin>
+          <param name="mock_sensor_commands">${mock_sensor_commands}</param>
+        </xacro:if>
       </hardware>
       <joint name="virtual_front_wheel_joint">
@@ -16,4 +21,9 @@
         <state_interface name="position"/>
       </joint>
+      <sensor name="imu_sensor">
+        <state_interface name="roll" />
+        <state_interface name="pitch" />
+        <state_interface name="yaw" />
+      </sensor>
     </ros2_control>
   </xacro:macro>
