Commit message: add ekf for sensor fusion

File: description/urdf/carlikebot.urdf.xacro (robot description, xacro)
@@ -5,4 +5,5 @@
   <xacro:arg name="mock_sensor_commands" default="false" />
   <xacro:arg name="use_gazebo_classic" default="false" />
+  <xacro:arg name="use_ekf" default="true" />
   <!-- <xacro:arg name="prefix" default="" /> -->
   <!-- Import carlikebot description -->
@@ -22,5 +23,6 @@
     <!-- Import Gazebo Classic definitions + plugin -->
     <xacro:include filename="carlikebot/carlikebot.gazebo.xacro" />
-    <xacro:carlikebot_gazebo />
+    <xacro:carlikebot_gazebo
+      use_ekf="$(arg use_ekf)" />
   </xacro:if>
 </robot>

File: description/urdf/carlikebot/carlikebot.gazebo.xacro (robot description, xacro)
@@ -5,5 +5,5 @@
 -->
 <robot xmlns:xacro="http://ros.org/wiki/xacro">
-  <xacro:macro name="carlikebot_gazebo">
+  <xacro:macro name="carlikebot_gazebo" params="use_ekf">
     <!-- ros_control plugin -->
     <gazebo>
@@ -11,7 +11,9 @@
         <parameters>$(find carlikebot_bringup)/config/carlikebot_controllers.yaml</parameters>
         <parameters>$(find carlikebot_bringup)/config/use_sim_time.yaml</parameters>
-        <ros>
-            <remapping>/bicycle_steering_controller/tf_odometry:=tf</remapping>
-        </ros>
+        <xacro:unless value="${use_ekf}">
+          <ros>
+              <remapping>/bicycle_steering_controller/tf_odometry:=tf</remapping>
+          </ros>
+        </xacro:unless>
       </plugin>
     </gazebo>

File: description/urdf/carlikebot/carlikebot.ros2_control.xacro (robot description, xacro)
@@ -18,8 +18,8 @@
         </command_interface>
         <state_interface name="position">
-          <param name="initial_value">0.0</param>
+          <!-- <param name="initial_value">0.0</param> -->
         </state_interface>
         <state_interface name="position">
-          <param name="initial_value">0.0</param>
+          <!-- <param name="initial_value">0.0</param> -->
         </state_interface>
       </joint>
@@ -30,8 +30,8 @@
         </command_interface>
         <state_interface name="velocity">
-          <param name="initial_value">0.0</param>
+          <!-- <param name="initial_value">0.0</param> -->
         </state_interface>
         <state_interface name="position">
-          <param name="initial_value">0.0</param>
+          <!-- <param name="initial_value">0.0</param> -->
         </state_interface>
       </joint>
