Commit message: add imu sensor

File: description/urdf/carlikebot/carlikebot.description.urdf.xacro (robot description, xacro)
@@ -45,4 +45,27 @@
       <axis xyz="0 0 1"/>
       <dynamics damping="0.2"/>
+    </joint>
+    <!-- IMU sensor -->
+    <link name="imu_link">
+      <visual>
+        <origin xyz="0 0 0" rpy="0 0 0"/>
+        <geometry>
+          <box size="0.0000001 0.0000001 0.0000001"/>
+        </geometry>
+        <material name="invisible"/>
+      </visual>
+      <inertial>
+        <origin xyz="0 0 0" rpy="0 0 0"/>
+        <mass value="0.0000001"/>
+          <inertia
+            ixx="0.0000001" ixy="0.0" ixz="0.0"
+            iyy="0.0000001" iyz="0.0"
+            izz="0.0000001"/>
+      </inertial>
+    </link>
+    <joint name="imu_joint" type="fixed">
+      <parent link="chassis_link"/>
+      <child link="imu_link"/>
+      <origin xyz="0 0 0" rpy="0 0 0"/>
     </joint>
     <!-- rear wheels -->

File: description/urdf/carlikebot/carlikebot.gazebo.xacro (robot description, xacro)
@@ -16,4 +16,15 @@
       </plugin>
     </gazebo>
+  <gazebo reference="imu_link">
+    <sensor name="imu_sensor" type="imu">
+      <always_on>true</always_on>
+      <update_rate>100</update_rate>
+      <plugin filename="libgazebo_ros_imu_sensor.so" name="imu_plugin">
+          <ros>
+            <remapping>~/out:=imu</remapping>
+          </ros>
+      </plugin>
+    </sensor>
+  </gazebo>
   </xacro:macro>
 </robot>

File: description/urdf/carlikebot/carlikebot.ros2_control.xacro (robot description, xacro)
@@ -36,12 +36,16 @@
         </state_interface>
       </joint>
-      <!-- <sensor name="imu_sensor">
-        <state_interface name="roll" />
-        <state_interface name="pitch" />
-        <state_interface name="yaw" />
-        <state_interface name="orientation.x" />
-        <state_interface name="angular_velocity.x" />
-        <state_interface name="linear_acceleration.x" />
-      </sensor> -->
+      <sensor name="imu_sensor">
+        <state_interface name="orientation.x"/>
+        <state_interface name="orientation.y"/>
+        <state_interface name="orientation.z"/>
+        <state_interface name="orientation.w"/>
+        <state_interface name="angular_velocity.x"/>
+        <state_interface name="angular_velocity.y"/>
+        <state_interface name="angular_velocity.z"/>
+        <state_interface name="linear_acceleration.x"/>
+        <state_interface name="linear_acceleration.y"/>
+        <state_interface name="linear_acceleration.z"/>
+      </sensor>
     </ros2_control>
   </xacro:macro>

Commit message: add ultrasonic sensor and world

File: description/urdf/carlikebot/carlikebot.description.urdf.xacro (robot description, xacro)
@@ -68,4 +68,27 @@
       <child link="imu_link"/>
       <origin xyz="0 0 0" rpy="0 0 0"/>
+    </joint>
+    <!-- Ultrasonic sensor -->
+    <link name="ultrasonic_link">
+      <visual>
+        <origin xyz="0.001 0.001 0.001" rpy="0 0 0"/>
+        <geometry>
+          <box size="0.0000001 0.0000001 0.0000001"/>
+        </geometry>
+        <material name="invisible"/>
+      </visual>
+      <inertial>
+        <origin xyz="0 0 0" rpy="0 0 0"/>
+        <mass value="0.0000001"/>
+          <inertia
+            ixx="0.0000001" ixy="0.0" ixz="0.0"
+            iyy="0.0000001" iyz="0.0"
+            izz="0.0000001"/>
+      </inertial>
+    </link>
+    <joint name="ultrasonic_joint" type="fixed">
+      <parent link="chassis_link"/>
+      <child link="ultrasonic_link"/>
+      <origin xyz="0.0 0.0 0.12" rpy="0 0 0"/>
     </joint>
     <!-- rear wheels -->

File: description/urdf/carlikebot/carlikebot.gazebo.xacro (robot description, xacro)
@@ -24,4 +24,45 @@
       </sensor>
     </gazebo>
+    <gazebo reference="ultrasonic_link">
+      <sensor name="ultrasonic" type="ray">
+        <always_on>true</always_on>
+        <visualize>true</visualize>
+        <update_rate>5</update_rate>
+        <ray>
+          <scan>
+            <horizontal>
+              <samples>5</samples>
+              <resolution>1.000000</resolution>
+              <min_angle>-0.12</min_angle>
+              <max_angle>0.12</max_angle>
+            </horizontal>
+            <vertical>
+              <samples>5</samples>
+              <resolution>1.000000</resolution>
+              <min_angle>-0.01</min_angle>
+              <max_angle>0.01</max_angle>
+            </vertical>
+          </scan>
+          <range>
+            <min>0.02</min>
+            <max>4</max>
+            <resolution>0.01</resolution>
+          </range>
+          <noise>
+            <type>gaussian</type>
+            <mean>0.0</mean>
+            <stddev>0.01</stddev>
+          </noise>
+        </ray>
+        <plugin name="ultrasonic_sensor" filename="libgazebo_ros_ray_sensor.so">
+          <ros>
+            <remapping>~/out:=scan</remapping>
+          </ros>
+          <output_type>sensor_msgs/Range</output_type>
+          <radiation_type>ultrasound</radiation_type>
+          <frame_name>ultrasonic_link</frame_name>
+        </plugin>
+      </sensor>
+    </gazebo>
   </xacro:macro>
 </robot>

Commit message: add camera sensor

File: description/urdf/carlikebot/carlikebot.description.urdf.xacro (robot description, xacro)
@@ -92,4 +92,27 @@
       <origin xyz="0.0 0.0 0.12" rpy="0 0 0"/>
     </joint>
+    <!-- Camera sensor -->
+    <link name="camera_link">
+      <visual>
+        <origin xyz="0.002 0.002 0.002" rpy="0 0 0"/>
+        <geometry>
+          <box size="0.0000001 0.0000001 0.0000001"/>
+        </geometry>
+        <material name="invisible"/>
+      </visual>
+      <inertial>
+        <origin xyz="0 0 0" rpy="0 0 0"/>
+        <mass value="0.0000001"/>
+          <inertia
+            ixx="0.0000001" ixy="0.0" ixz="0.0"
+            iyy="0.0000001" iyz="0.0"
+            izz="0.0000001"/>
+      </inertial>
+    </link>
+    <joint name="camera_joint" type="fixed">
+      <parent link="chassis_link"/>
+      <child link="camera_link"/>
+      <origin xyz="0.0 0.0 0.2" rpy="0 0 0"/>
+    </joint>
     <!-- rear wheels -->
     <!-- virtual rear wheel -->

File: description/urdf/carlikebot/carlikebot.gazebo.xacro (robot description, xacro)
@@ -65,4 +65,28 @@
       </sensor>
     </gazebo>
+    <gazebo reference="camera_link">
+      <sensor type="camera" name="picamera">
+        <always_on>1</always_on>
+        <update_rate>30</update_rate>
+        <visualize>true</visualize>
+        <camera>
+          <horizontal_fov>1.047</horizontal_fov>
+          <image>
+            <width>320</width>
+            <height>240</height>
+          </image>
+          <clip>
+            <near>0.1</near>
+            <far>100</far>
+          </clip>
+        </camera>
+        <plugin name="camera_controller" filename="libgazebo_ros_camera.so">
+          <baseline>0.2</baseline>
+          <alwaysOn>true</alwaysOn>
+          <updateRate>0.0</updateRate>
+          <frame_name>camera_link</frame_name>
+        </plugin>
+      </sensor>
+    </gazebo>
   </xacro:macro>
 </robot>
