Commit message: add lidar and navigation package

File: carlikebot_description/urdf/carlikebot/carlikebot.description.urdf.xacro (robot description, xacro)
@@ -15,4 +15,11 @@
   <!-- Base Link -->
   <link name="base_link" />
+  <!--Base footprint link (it's for slam)-->
+  <link name="base_footprint" />
+  <joint name="base_footprint_joint" type="fixed">
+    <parent link="base_link"/>
+    <child link="base_footprint"/>
+    <origin xyz="0 0 0" rpy="0 0 0"/>
+  </joint>
   <!-- Chassis -->
   <link name="chassis_link">
@@ -70,5 +77,5 @@
     </joint>
     <!-- Ultrasonic sensor -->
-    <link name="ultrasonic_link">
+    <!-- <link name="ultrasonic_link">
       <visual>
         <origin xyz="0.001 0.001 0.001" rpy="0 0 0"/>
@@ -91,7 +98,7 @@
       <child link="ultrasonic_link"/>
       <origin xyz="0.0 0.0 0.12" rpy="0 0 0"/>
-    </joint>
+    </joint> -->
     <!-- Camera sensor -->
-    <link name="camera_link">
+    <!-- <link name="camera_link">
       <visual>
         <origin xyz="0.002 0.002 0.002" rpy="0 0 0"/>
@@ -114,4 +121,23 @@
       <child link="camera_link"/>
       <origin xyz="0.0 0.0 0.2" rpy="0 0 0"/>
+    </joint> -->
+    <!-- Lidar sensor -->
+    <link name="lidar_link">
+      <inertial>
+        <origin xyz="0 0 0" rpy="0 0 0"/>
+        <mass value="0.125"/>
+        <inertia ixx="0.001"  ixy="0"  ixz="0" iyy="0.001" iyz="0" izz="0.001" />
+      </inertial>
+      <visual>
+        <origin xyz="0 0 0" rpy="0 0 0"/>
+        <geometry>
+          <cylinder radius="0.0508" length="0.055"/>
+        </geometry>
+      </visual>
+    </link>
+    <joint name="lidar_joint" type="fixed">
+      <parent link="chassis_link"/>
+      <child link="lidar_link"/>
+      <origin xyz="0 0 0.12" rpy="0 0 0"/>
     </joint>
     <!-- rear wheels -->

File: carlikebot_description/urdf/carlikebot/carlikebot.gazebo.xacro (robot description, xacro)
@@ -24,5 +24,5 @@
       </sensor>
     </gazebo>
-    <gazebo reference="ultrasonic_link">
+    <!-- <gazebo reference="ultrasonic_link">
       <sensor name="ultrasonic" type="ray">
         <always_on>true</always_on>
@@ -57,5 +57,5 @@
         <plugin name="ultrasonic_sensor" filename="libgazebo_ros_ray_sensor.so">
           <ros>
-            <remapping>~/out:=scan</remapping>
+            <remapping>~/out:=range_scan</remapping>
           </ros>
           <output_type>sensor_msgs/Range</output_type>
@@ -64,6 +64,6 @@
         </plugin>
       </sensor>
-    </gazebo>
-    <gazebo reference="camera_link">
+    </gazebo> -->
+    <!-- <gazebo reference="camera_link">
       <sensor type="camera" name="picamera">
         <always_on>1</always_on>
@@ -87,4 +87,38 @@
         </plugin>
       </sensor>
+    </gazebo> -->
+    <gazebo reference="lidar_link">
+      <sensor name="lidar" type="ray">
+        <always_on>true</always_on>
+        <visualize>true</visualize>
+        <update_rate>5</update_rate>
+        <ray>
+          <scan>
+            <horizontal>
+              <samples>360</samples>
+              <resolution>1.000000</resolution>
+              <min_angle>0.000000</min_angle>
+              <max_angle>6.280000</max_angle>
+            </horizontal>
+          </scan>
+          <range>
+            <min>0.120000</min>
+            <max>3.5</max>
+            <resolution>0.015000</resolution>
+          </range>
+          <noise>
+            <type>gaussian</type>
+            <mean>0.0</mean>
+            <stddev>0.01</stddev>
+          </noise>
+        </ray>
+        <plugin name="scan" filename="libgazebo_ros_ray_sensor.so">
+          <ros>
+            <remapping>~/out:=scan</remapping>
+          </ros>
+          <output_type>sensor_msgs/LaserScan</output_type>
+          <frame_name>lidar_link</frame_name>
+        </plugin>
+      </sensor>
     </gazebo>
   </xacro:macro>

Commit message: remap topic and tweek urdf a bit

File: carlikebot_description/urdf/carlikebot/carlikebot.description.urdf.xacro (robot description, xacro)
@@ -24,10 +24,10 @@
   <!-- Chassis -->
   <link name="chassis_link">
-    <collision>
+    <!-- <collision>
       <origin xyz="0 0 0" rpy="0 0 0"/>
       <geometry>
         <box size="${base_length} ${base_width} ${base_height}"/>
       </geometry>
-    </collision>
+    </collision> -->
     <visual>
       <origin xyz="0 0 0" rpy="0 0 0"/>
@@ -144,10 +144,16 @@
     <!-- virtual rear wheel -->
     <link name="virtual_rear_wheel">
-      <visual>
+      <collision>
         <origin xyz="0 0 0" rpy="${PI/2} 0 ${PI/2}"/>
         <geometry>
           <cylinder length="0.01" radius="${wheel_radius}"/>
         </geometry>
-        <material name="invisible"/>
+      </collision>
+      <visual>
+        <origin xyz="0 0 0" rpy="${PI/2} 0 ${PI/2}"/>
+        <geometry>
+          <cylinder length="0.01" radius="${wheel_radius}"/>
+        </geometry>
+        <material name="black"/>
       </visual>
       <inertial>
@@ -166,5 +172,5 @@
       <axis xyz="1 0 0"/>
       <limit effort="100.0" velocity="100.0"/>
-      <dynamics damping="0.2"/>
+      <!-- <dynamics damping="0.2"/> -->
     </joint>
     <!-- rear right wheel -->
@@ -198,5 +204,5 @@
       <axis xyz="1 0 0"/>
       <limit effort="100.0" velocity="100.0"/>
-      <dynamics damping="0.2"/>
+      <!-- <dynamics damping="0.2"/> -->
       <mimic joint="virtual_rear_wheel_joint" multiplier="1.0" offset="0.0"/>
     </joint>
@@ -231,5 +237,5 @@
       <axis xyz="1 0 0"/>
       <limit effort="100.0" velocity="100.0"/>
-      <dynamics damping="0.2"/>
+      <!-- <dynamics damping="0.2"/> -->
       <mimic joint="virtual_rear_wheel_joint" multiplier="1.0" offset="0.0"/>
     </joint>
@@ -237,10 +243,16 @@
     <!-- virtual front wheel -->
     <link name="virtual_front_wheel">
-      <visual>
+      <collision>
         <origin xyz="0 0 0" rpy="${PI/2} 0 ${PI/2}"/>
         <geometry>
           <cylinder length="0.01" radius="${wheel_radius}"/>
         </geometry>
-        <material name="invisible"/>
+      </collision>
+      <visual>
+        <origin xyz="0 0 0" rpy="${PI/2} 0 ${PI/2}"/>
+        <geometry>
+          <cylinder length="0.01" radius="${wheel_radius}"/>
+        </geometry>
+        <material name="black"/>
       </visual>
       <inertial>
@@ -254,10 +266,12 @@
     </link>
     <joint name="virtual_front_wheel_joint" type="revolute">
+    <!-- <joint name="virtual_front_wheel_joint" type="continuous"> -->
       <parent link="chassis_link"/>
       <child link="virtual_front_wheel"/>
       <origin xyz="${wheelbase/2} 0 -${base_height/2}" rpy="0 0 ${PI/2}"/>
       <axis xyz="0 0 1"/>
+      <!-- <limit effort="100.0" velocity="100.0"/> -->
       <limit lower="-0.4" upper="0.4" effort="100.0" velocity="0.0"/>
-      <dynamics damping="0.2"/>
+      <!-- <dynamics damping="0.2"/> -->
     </joint>
     <!-- front right wheel -->
@@ -286,10 +300,12 @@
     </link>
     <joint name="front_right_wheel_joint" type="revolute">
+    <!-- <joint name="front_right_wheel_joint" type="continuous"> -->
       <parent link="chassis_link" />
       <child link="front_right_wheel" />
       <origin xyz="${wheelbase/2} ${base_width/2} -${base_height/2}" rpy="0 0 ${PI/2}"/>
       <axis xyz="0 0 1"/>
+      <!-- <limit effort="100.0" velocity="100.0"/> -->
       <limit lower="-0.4" upper="0.4" effort="100.0" velocity="0.0"/>
-      <dynamics damping="0.2"/>
+      <!-- <dynamics damping="0.2"/> -->
       <mimic joint="virtual_front_wheel_joint" multiplier="1.0" offset="0.0"/>
     </joint>
@@ -319,10 +335,12 @@
     </link>
     <joint name="front_left_wheel_joint" type="revolute">
+    <!-- <joint name="front_left_wheel_joint" type="continuous"> -->
       <parent link="chassis_link" />
       <child link="front_left_wheel" />
       <origin xyz="${wheelbase/2} -${base_width/2} -${base_height/2}" rpy="0 0 ${PI/2}"/>
       <axis xyz="0 0 1"/>
+      <!-- <limit effort="100.0" velocity="100.0"/> -->
       <limit lower="-0.4" upper="0.4" effort="100.0" velocity="0.0"/>
-      <dynamics damping="0.2"/>
+      <!-- <dynamics damping="0.2"/> -->
       <mimic joint="virtual_front_wheel_joint" multiplier="1.0" offset="0.0"/>
     </joint>

Commit message: change urdf values to real life ones

File: carlikebot_description/urdf/carlikebot/carlikebot.description.urdf.xacro (robot description, xacro)
@@ -2,46 +2,50 @@
 <robot xmlns:xacro="http://www.ros.org/wiki/xacro">
   <xacro:macro name="carlikebot">
-  <!-- Constants for robot dimensions -->
-  <xacro:property name="PI" value="3.1415926535897931"/>
-  <xacro:property name="base_mass" value="4.0" /> <!-- arbitrary value for base mass -->
-  <xacro:property name="base_width" value="0.260" />
-  <xacro:property name="base_length" value="0.525" />
-  <xacro:property name="base_height" value="0.060" />
-  <xacro:property name="wheelbase" value="0.325" />
-  <xacro:property name="wheel_mass" value="0.34055" /> <!-- arbitrary value for wheel mass -->
-  <xacro:property name="wheel_len" value="0.045" />
-  <xacro:property name="wheel_radius" value="0.05" />
-  <!-- <xacro:property name="wheeltrack" value="" -->
-  <!-- Base Link -->
-  <link name="base_link" />
-  <!--Base footprint link (it's for slam)-->
-  <link name="base_footprint" />
-  <joint name="base_footprint_joint" type="fixed">
-    <parent link="base_link"/>
-    <child link="base_footprint"/>
-    <origin xyz="0 0 0" rpy="0 0 0"/>
-  </joint>
-  <!-- Chassis -->
-  <link name="chassis_link">
-    <!-- <collision>
+    <!-- Constants for robot dimensions -->
+    <xacro:property name="PI" value="3.1415926535897931"/>
+    <xacro:property name="base_mass" value="4.0" /> <!-- arbitrary value for base mass -->
+    <xacro:property name="base_width" value="0.09" />
+    <xacro:property name="base_length" value="0.195" />
+    <xacro:property name="base_height" value="0.002" />
+    <xacro:property name="wheelbase" value="0.145" />
+    <xacro:property name="wheel_mass" value="0.34055" /> <!-- arbitrary value for wheel mass -->
+    <xacro:property name="wheel_len" value="0.025" />
+    <xacro:property name="wheel_radius" value="0.0325" />
+    <xacro:property name="wheel_ygap" value="0.005"/>
+    <xacro:property name="wheel_zoff" value="0.0125"/>
+    <xacro:property name="wheel_back_xoff" value="0.0775"/>
+    <xacro:property name="wheel_front_xoff" value="0.065"/>
+    <!-- <xacro:property name="wheeltrack" value="" -->
+    <!-- Base Link -->
+    <link name="base_link" />
+    <!--Base footprint link (it's for slam)-->
+    <link name="base_footprint" />
+    <joint name="base_footprint_joint" type="fixed">
+      <parent link="base_link"/>
+      <child link="base_footprint"/>
       <origin xyz="0 0 0" rpy="0 0 0"/>
-      <geometry>
-        <box size="${base_length} ${base_width} ${base_height}"/>
-      </geometry>
-    </collision> -->
-    <visual>
-      <origin xyz="0 0 0" rpy="0 0 0"/>
-      <geometry>
-        <box size="${base_length} ${base_width} ${base_height}"/>
-      </geometry>
-      <material name="orange"/>
-    </visual>
-    <inertial>
-      <origin xyz="0 0 0" rpy="0 0 0"/>
-      <mass value="${base_mass}"/>
-        <inertia
-          ixx="0.000270" ixy="0.0" ixz="0.0"
-          iyy="0.000270" iyz="0.0"
-          izz="0.000426"/>
+    </joint>
+    <!-- Chassis -->
+    <link name="chassis_link">
+      <!-- <collision>
+        <origin xyz="0 0 0" rpy="0 0 0"/>
+        <geometry>
+          <box size="${base_length} ${base_width} ${base_height}"/>
+        </geometry>
+      </collision> -->
+      <visual>
+        <origin xyz="0 0 0" rpy="0 0 0"/>
+        <geometry>
+          <box size="${base_length} ${base_width} ${base_height}"/>
+        </geometry>
+        <material name="orange"/>
+      </visual>
+      <inertial>
+        <origin xyz="0 0 0" rpy="0 0 0"/>
+        <mass value="${base_mass}"/>
+          <inertia
+            ixx="0.000292419" ixy="0.0" ixz="0.0"
+            iyy="0.001372213" iyz="0.0"
+            izz="0.00166434375"/>
       </inertial>
     </link>
@@ -127,10 +131,10 @@
         <origin xyz="0 0 0" rpy="0 0 0"/>
         <mass value="0.125"/>
-        <inertia ixx="0.001"  ixy="0"  ixz="0" iyy="0.001" iyz="0" izz="0.001" />
-      </inertial>
-      <visual>
-        <origin xyz="0 0 0" rpy="0 0 0"/>
-        <geometry>
-          <cylinder radius="0.0508" length="0.055"/>
+        <inertia ixx="0.000001"  ixy="0"  ixz="0" iyy="0.000001" iyz="0" izz="0.000001" />
+      </inertial>
+      <visual>
+        <origin xyz="0 0 0" rpy="0 0 0"/>
+        <geometry>
+          <cylinder radius="0.01" length="0.01"/>
         </geometry>
       </visual>
@@ -147,21 +151,21 @@
         <origin xyz="0 0 0" rpy="${PI/2} 0 ${PI/2}"/>
         <geometry>
-          <cylinder length="0.01" radius="${wheel_radius}"/>
-        </geometry>
-      </collision>
-      <visual>
-        <origin xyz="0 0 0" rpy="${PI/2} 0 ${PI/2}"/>
-        <geometry>
-          <cylinder length="0.01" radius="${wheel_radius}"/>
-        </geometry>
-        <material name="black"/>
-      </visual>
-      <inertial>
-        <origin xyz="0 0 0" rpy="${PI/2} 0 ${PI/2}"/>
-        <mass value="${wheel_mass}"/>
-        <inertia
-          ixx="0.000270" ixy="0.0" ixz="0.0"
-          iyy="0.000270" iyz="0.0"
-          izz="0.000426"/>
+          <cylinder length="${wheel_len}" radius="${wheel_radius}"/>
+        </geometry>
+      </collision>
+      <visual>
+        <origin xyz="0 0 0" rpy="${PI/2} 0 ${PI/2}"/>
+        <geometry>
+          <cylinder length="${wheel_len}" radius="${wheel_radius}"/>
+        </geometry>
+        <material name="invisible"/>
+      </visual>
+      <inertial>
+        <origin xyz="0 0 0" rpy="${PI/2} 0 ${PI/2}"/>
+        <mass value="${wheel_mass}"/>
+        <inertia
+          ixx="0.0000075875" ixy="0.0" ixz="0.0"
+          iyy="0.0000075875" iyz="0.0"
+          izz="0.000012675"/>
       </inertial>
     </link>
@@ -169,5 +173,5 @@
       <parent link="chassis_link"/>
       <child link="virtual_rear_wheel"/>
-      <origin xyz="-${wheelbase/2} 0 -${base_height/2}" rpy="0 0 ${PI/2}"/>
+      <origin xyz="-${wheel_back_xoff} 0 -${wheel_zoff}" rpy="0 0 ${PI/2}"/>
       <axis xyz="1 0 0"/>
       <limit effort="100.0" velocity="100.0"/>
@@ -193,7 +197,7 @@
         <mass value="${wheel_mass}"/>
         <inertia
-          ixx="0.000270" ixy="0.0" ixz="0.0"
-          iyy="0.000270" iyz="0.0"
-          izz="0.000426"/>
+          ixx="0.0000075875" ixy="0.0" ixz="0.0"
+          iyy="0.0000075875" iyz="0.0"
+          izz="0.000012675"/>
       </inertial>
     </link>
@@ -201,5 +205,5 @@
       <parent link="chassis_link"/>
       <child link="rear_right_wheel"/>
-      <origin xyz="-${wheelbase/2} ${base_width/2} -${base_height/2}" rpy="0 0 ${PI/2}"/>
+      <origin xyz="-${wheel_back_xoff} -${base_width/2+wheel_ygap+wheel_len/2} -${wheel_zoff}" rpy="0 0 ${PI/2}"/>
       <axis xyz="1 0 0"/>
       <limit effort="100.0" velocity="100.0"/>
@@ -226,7 +230,7 @@
           <mass value="${wheel_mass}"/>
           <inertia
-            ixx="0.000270" ixy="0.0" ixz="0.0"
-            iyy="0.000270" iyz="0.0"
-            izz="0.000426"/>
+            ixx="0.0000075875" ixy="0.0" ixz="0.0"
+            iyy="0.0000075875" iyz="0.0"
+            izz="0.000012675"/>
         </inertial>
     </link>
@@ -234,5 +238,5 @@
       <parent link="chassis_link" />
       <child link="rear_left_wheel" />
-      <origin xyz="-${wheelbase/2} -${base_width/2} -${base_height/2}" rpy="0 0 ${PI/2}"/>
+      <origin xyz="-${wheel_back_xoff} ${base_width/2+wheel_ygap+wheel_len/2} -${wheel_zoff}" rpy="0 0 ${PI/2}"/>
       <axis xyz="1 0 0"/>
       <limit effort="100.0" velocity="100.0"/>
@@ -246,33 +250,41 @@
         <origin xyz="0 0 0" rpy="${PI/2} 0 ${PI/2}"/>
         <geometry>
-          <cylinder length="0.01" radius="${wheel_radius}"/>
-        </geometry>
-      </collision>
-      <visual>
-        <origin xyz="0 0 0" rpy="${PI/2} 0 ${PI/2}"/>
-        <geometry>
-          <cylinder length="0.01" radius="${wheel_radius}"/>
-        </geometry>
-        <material name="black"/>
-      </visual>
-      <inertial>
-        <origin xyz="0 0 0" rpy="${PI/2} 0 ${PI/2}"/>
-        <mass value="${wheel_mass}"/>
-        <inertia
-          ixx="0.000270" ixy="0.0" ixz="0.0"
-          iyy="0.000270" iyz="0.0"
-          izz="0.000426"/>
-      </inertial>
-    </link>
-    <joint name="virtual_front_wheel_joint" type="revolute">
-    <!-- <joint name="virtual_front_wheel_joint" type="continuous"> -->
+          <cylinder length="${wheel_len}" radius="${wheel_radius}"/>
+        </geometry>
+      </collision>
+      <visual>
+        <origin xyz="0 0 0" rpy="${PI/2} 0 ${PI/2}"/>
+        <geometry>
+          <cylinder length="${wheel_len}" radius="${wheel_radius}"/>
+        </geometry>
+        <material name="invisible"/>
+      </visual>
+      <inertial>
+        <origin xyz="0 0 0" rpy="${PI/2} 0 ${PI/2}"/>
+        <mass value="${wheel_mass}"/>
+        <inertia
+          ixx="0.0000075875" ixy="0.0" ixz="0.0"
+          iyy="0.0000075875" iyz="0.0"
+          izz="0.000012675"/>
+      </inertial>
+    </link>
+    <!-- <joint name="virtual_front_wheel_joint" type="revolute"> -->
+    <joint name="virtual_front_wheel_joint" type="continuous">
       <parent link="chassis_link"/>
       <child link="virtual_front_wheel"/>
-      <origin xyz="${wheelbase/2} 0 -${base_height/2}" rpy="0 0 ${PI/2}"/>
+      <origin xyz="${wheel_front_xoff} 0 -${wheel_zoff}" rpy="0 0 ${PI/2}"/>
+      <!-- <axis xyz="0 0 1"/> -->
+      <axis xyz="1 0 0"/>
+      <limit effort="100.0" velocity="100.0"/>
+      <!-- <limit lower="-0.4" upper="0.4" effort="100.0" velocity="0.0"/> -->
+      <!-- <dynamics damping="0.2"/> -->
+    </joint>
+    <!-- <joint name="virtual_front_wheel_steer_joint" type="revolute">
+      <parent link="chassis_link"/>
+      <child link="virtual_front_wheel"/>
+      <origin xyz="${wheel_front_xoff} 0 -${wheel_zoff}" rpy="0 0 ${PI/2}"/>
       <axis xyz="0 0 1"/>
-      <!-- <limit effort="100.0" velocity="100.0"/> -->
       <limit lower="-0.4" upper="0.4" effort="100.0" velocity="0.0"/>
-      <!-- <dynamics damping="0.2"/> -->
-    </joint>
+    </joint> -->
     <!-- front right wheel -->
     <link name="front_right_wheel">
@@ -294,20 +306,29 @@
         <mass value="${wheel_mass}"/>
         <inertia
-          ixx="0.000270" ixy="0.0" ixz="0.0"
-          iyy="0.000270" iyz="0.0"
-          izz="0.000426"/>
-      </inertial>
-    </link>
-    <joint name="front_right_wheel_joint" type="revolute">
-    <!-- <joint name="front_right_wheel_joint" type="continuous"> -->
+          ixx="0.0000075875" ixy="0.0" ixz="0.0"
+          iyy="0.0000075875" iyz="0.0"
+          izz="0.000012675"/>
+      </inertial>
+    </link>
+    <!-- <joint name="front_right_wheel_joint" type="revolute"> -->
+    <joint name="front_right_wheel_joint" type="continuous">
       <parent link="chassis_link" />
       <child link="front_right_wheel" />
-      <origin xyz="${wheelbase/2} ${base_width/2} -${base_height/2}" rpy="0 0 ${PI/2}"/>
+      <origin xyz="${wheel_front_xoff} -${base_width/2+wheel_ygap+wheel_len/2} -${wheel_zoff}" rpy="0 0 ${PI/2}"/>
+      <!-- <axis xyz="0 0 1"/> -->
+            <axis xyz="1 0 0"/>
+      <limit effort="100.0" velocity="100.0"/>
+      <!-- <limit lower="-0.4" upper="0.4" effort="100.0" velocity="0.0"/> -->
+      <!-- <dynamics damping="0.2"/> -->
+      <mimic joint="virtual_front_wheel_joint" multiplier="1.0" offset="0.0"/>
+    </joint>
+    <!-- <joint name="front_right_wheel_steer_joint" type="revolute">
+      <parent link="chassis_link" />
+      <child link="front_right_wheel" />
+      <origin xyz="${wheel_front_xoff} -${base_width/2+wheel_ygap+wheel_len/2} -${wheel_zoff}" rpy="0 0 ${PI/2}"/>
       <axis xyz="0 0 1"/>
-      <!-- <limit effort="100.0" velocity="100.0"/> -->
       <limit lower="-0.4" upper="0.4" effort="100.0" velocity="0.0"/>
-      <!-- <dynamics damping="0.2"/> -->
-      <mimic joint="virtual_front_wheel_joint" multiplier="1.0" offset="0.0"/>
-    </joint>
+      <mimic joint="virtual_front_wheel_steer_joint" multiplier="1.0" offset="0.0"/>
+    </joint> -->
     <!-- front left steering -->
     <link name="front_left_wheel">
@@ -329,20 +350,29 @@
         <mass value="${wheel_mass}"/>
         <inertia
-          ixx="0.000270" ixy="0.0" ixz="0.0"
-          iyy="0.000270" iyz="0.0"
-          izz="0.000426"/>
-      </inertial>
-    </link>
-    <joint name="front_left_wheel_joint" type="revolute">
-    <!-- <joint name="front_left_wheel_joint" type="continuous"> -->
+          ixx="0.0000075875" ixy="0.0" ixz="0.0"
+          iyy="0.0000075875" iyz="0.0"
+          izz="0.000012675"/>
+      </inertial>
+    </link>
+    <!-- <joint name="front_left_wheel_joint" type="revolute"> -->
+    <joint name="front_left_wheel_joint" type="continuous">
       <parent link="chassis_link" />
       <child link="front_left_wheel" />
-      <origin xyz="${wheelbase/2} -${base_width/2} -${base_height/2}" rpy="0 0 ${PI/2}"/>
+      <origin xyz="${wheel_front_xoff} ${base_width/2+wheel_ygap+wheel_len/2} -${wheel_zoff}" rpy="0 0 ${PI/2}"/>
+      <!-- <axis xyz="0 0 1"/> -->
+      <axis xyz="1 0 0"/>
+      <limit effort="100.0" velocity="100.0"/>
+      <!-- <limit lower="-0.4" upper="0.4" effort="100.0" velocity="0.0"/> -->
+      <!-- <dynamics damping="0.2"/> -->
+      <mimic joint="virtual_front_wheel_joint" multiplier="1.0" offset="0.0"/>
+    </joint>
+    <!-- <joint name="front_left_wheel_steer_joint" type="revolute">
+      <parent link="chassis_link" />
+      <child link="front_left_wheel" />
+      <origin xyz="${wheel_front_xoff} ${base_width/2+wheel_ygap+wheel_len/2} -${wheel_zoff}" rpy="0 0 ${PI/2}"/>
       <axis xyz="0 0 1"/>
-      <!-- <limit effort="100.0" velocity="100.0"/> -->
       <limit lower="-0.4" upper="0.4" effort="100.0" velocity="0.0"/>
-      <!-- <dynamics damping="0.2"/> -->
-      <mimic joint="virtual_front_wheel_joint" multiplier="1.0" offset="0.0"/>
-    </joint>
+      <mimic joint="virtual_front_wheel_steer_joint" multiplier="1.0" offset="0.0"/>
+    </joint> -->
   </xacro:macro>
 </robot>

File: carlikebot_description/urdf/carlikebot/carlikebot.ros2_control.xacro (robot description, xacro)
@@ -14,11 +14,11 @@
       <joint name="virtual_front_wheel_joint">
         <command_interface name="position">
-          <param name="min">-100</param>
-          <param name="max">100</param>
+          <param name="min">-10</param>
+          <param name="max">10</param>
         </command_interface>
         <state_interface name="position">
           <!-- <param name="initial_value">0.0</param> -->
         </state_interface>
-        <state_interface name="position">
+        <state_interface name="velocity">
           <!-- <param name="initial_value">0.0</param> -->
         </state_interface>
