Commit message: make virtual front wheel joint steer

File: carlikebot_description/urdf/carlikebot/carlikebot.description.urdf.xacro (robot description, xacro)
@@ -4,10 +4,10 @@
     <!-- Constants for robot dimensions -->
     <xacro:property name="PI" value="3.1415926535897931"/>
-    <xacro:property name="base_mass" value="4.0" /> <!-- arbitrary value for base mass -->
+    <xacro:property name="base_mass" value="0.433" /> <!-- arbitrary value for base mass, I think in Kg -->
     <xacro:property name="base_width" value="0.09" />
     <xacro:property name="base_length" value="0.195" />
     <xacro:property name="base_height" value="0.002" />
     <xacro:property name="wheelbase" value="0.145" />
-    <xacro:property name="wheel_mass" value="0.34055" /> <!-- arbitrary value for wheel mass -->
+    <xacro:property name="wheel_mass" value="0.024" /> <!-- arbitrary value for wheel mass, I think in Kg -->
     <xacro:property name="wheel_len" value="0.025" />
     <xacro:property name="wheel_radius" value="0.0325" />
@@ -269,16 +269,5 @@
       </inertial>
     </link>
-    <!-- <joint name="virtual_front_wheel_joint" type="revolute"> -->
-    <joint name="virtual_front_wheel_joint" type="continuous">
-      <parent link="chassis_link"/>
-      <child link="virtual_front_wheel"/>
-      <origin xyz="${wheel_front_xoff} 0 -${wheel_zoff}" rpy="0 0 ${PI/2}"/>
-      <!-- <axis xyz="0 0 1"/> -->
-      <axis xyz="1 0 0"/>
-      <limit effort="100.0" velocity="100.0"/>
-      <!-- <limit lower="-0.4" upper="0.4" effort="100.0" velocity="0.0"/> -->
-      <!-- <dynamics damping="0.2"/> -->
-    </joint>
-    <!-- <joint name="virtual_front_wheel_steer_joint" type="revolute">
+    <joint name="virtual_front_wheel_joint" type="revolute">
       <parent link="chassis_link"/>
       <child link="virtual_front_wheel"/>
@@ -286,5 +275,5 @@
       <axis xyz="0 0 1"/>
       <limit lower="-0.4" upper="0.4" effort="100.0" velocity="0.0"/>
-    </joint> -->
+    </joint>
     <!-- front right wheel -->
     <link name="front_right_wheel">
@@ -311,24 +300,12 @@
       </inertial>
     </link>
-    <!-- <joint name="front_right_wheel_joint" type="revolute"> -->
     <joint name="front_right_wheel_joint" type="continuous">
       <parent link="chassis_link" />
       <child link="front_right_wheel" />
       <origin xyz="${wheel_front_xoff} -${base_width/2+wheel_ygap+wheel_len/2} -${wheel_zoff}" rpy="0 0 ${PI/2}"/>
-      <!-- <axis xyz="0 0 1"/> -->
-            <axis xyz="1 0 0"/>
-      <limit effort="100.0" velocity="100.0"/>
-      <!-- <limit lower="-0.4" upper="0.4" effort="100.0" velocity="0.0"/> -->
-      <!-- <dynamics damping="0.2"/> -->
+      <axis xyz="1 0 0"/>
+      <limit effort="100.0" velocity="100.0"/>
       <mimic joint="virtual_front_wheel_joint" multiplier="1.0" offset="0.0"/>
     </joint>
-    <!-- <joint name="front_right_wheel_steer_joint" type="revolute">
-      <parent link="chassis_link" />
-      <child link="front_right_wheel" />
-      <origin xyz="${wheel_front_xoff} -${base_width/2+wheel_ygap+wheel_len/2} -${wheel_zoff}" rpy="0 0 ${PI/2}"/>
-      <axis xyz="0 0 1"/>
-      <limit lower="-0.4" upper="0.4" effort="100.0" velocity="0.0"/>
-      <mimic joint="virtual_front_wheel_steer_joint" multiplier="1.0" offset="0.0"/>
-    </joint> -->
     <!-- front left steering -->
     <link name="front_left_wheel">
@@ -355,24 +332,12 @@
       </inertial>
     </link>
-    <!-- <joint name="front_left_wheel_joint" type="revolute"> -->
     <joint name="front_left_wheel_joint" type="continuous">
       <parent link="chassis_link" />
       <child link="front_left_wheel" />
       <origin xyz="${wheel_front_xoff} ${base_width/2+wheel_ygap+wheel_len/2} -${wheel_zoff}" rpy="0 0 ${PI/2}"/>
-      <!-- <axis xyz="0 0 1"/> -->
-      <axis xyz="1 0 0"/>
-      <limit effort="100.0" velocity="100.0"/>
-      <!-- <limit lower="-0.4" upper="0.4" effort="100.0" velocity="0.0"/> -->
-      <!-- <dynamics damping="0.2"/> -->
+      <axis xyz="1 0 0"/>
+      <limit effort="100.0" velocity="100.0"/>
       <mimic joint="virtual_front_wheel_joint" multiplier="1.0" offset="0.0"/>
     </joint>
-    <!-- <joint name="front_left_wheel_steer_joint" type="revolute">
-      <parent link="chassis_link" />
-      <child link="front_left_wheel" />
-      <origin xyz="${wheel_front_xoff} ${base_width/2+wheel_ygap+wheel_len/2} -${wheel_zoff}" rpy="0 0 ${PI/2}"/>
-      <axis xyz="0 0 1"/>
-      <limit lower="-0.4" upper="0.4" effort="100.0" velocity="0.0"/>
-      <mimic joint="virtual_front_wheel_steer_joint" multiplier="1.0" offset="0.0"/>
-    </joint> -->
   </xacro:macro>
 </robot>

Commit message: fix ackerman steering

File: carlikebot_description/urdf/carlikebot/carlikebot.description.urdf.xacro (robot description, xacro)
@@ -247,10 +247,10 @@
     <!-- virtual front wheel -->
     <link name="virtual_front_wheel">
-      <collision>
-        <origin xyz="0 0 0" rpy="${PI/2} 0 ${PI/2}"/>
-        <geometry>
-          <cylinder length="${wheel_len}" radius="${wheel_radius}"/>
-        </geometry>
-      </collision>
+      <!-- <collision>
+        <origin xyz="0 0 0" rpy="${PI/2} 0 ${PI/2}"/>
+        <geometry>
+          <cylinder length="${wheel_len}" radius="${wheel_radius}"/>
+        </geometry>
+      </collision> -->
       <visual>
         <origin xyz="0 0 0" rpy="${PI/2} 0 ${PI/2}"/>
@@ -301,7 +301,9 @@
     </link>
     <joint name="front_right_wheel_joint" type="continuous">
-      <parent link="chassis_link" />
+      <!-- <parent link="chassis_link" /> -->
+      <parent link="virtual_front_wheel" />
       <child link="front_right_wheel" />
-      <origin xyz="${wheel_front_xoff} -${base_width/2+wheel_ygap+wheel_len/2} -${wheel_zoff}" rpy="0 0 ${PI/2}"/>
+      <!-- <origin xyz="${wheel_front_xoff} -${base_width/2+wheel_ygap+wheel_len/2} -${wheel_zoff}" rpy="0 0 ${PI/2}"/> -->
+      <origin xyz="-${base_width/2+wheel_ygap+wheel_len/2} 0 0" rpy="0 0 0"/>
       <axis xyz="1 0 0"/>
       <limit effort="100.0" velocity="100.0"/>
@@ -333,7 +335,9 @@
     </link>
     <joint name="front_left_wheel_joint" type="continuous">
-      <parent link="chassis_link" />
+      <!-- <parent link="chassis_link" /> -->
+      <parent link="virtual_front_wheel" />
       <child link="front_left_wheel" />
-      <origin xyz="${wheel_front_xoff} ${base_width/2+wheel_ygap+wheel_len/2} -${wheel_zoff}" rpy="0 0 ${PI/2}"/>
+      <!-- <origin xyz="${wheel_front_xoff} ${base_width/2+wheel_ygap+wheel_len/2} -${wheel_zoff}" rpy="0 0 ${PI/2}"/> -->
+      <origin xyz="${base_width/2+wheel_ygap+wheel_len/2} 0 0" rpy="0 0 0"/>
       <axis xyz="1 0 0"/>
       <limit effort="100.0" velocity="100.0"/>

Commit message: fix imu visualization and add friction

File: carlikebot_description/urdf/carlikebot/carlikebot.description.urdf.xacro (robot description, xacro)
@@ -55,5 +55,5 @@
       <origin xyz="0 0 ${base_height/2 + wheel_radius}" rpy="0 0 0"/>
       <axis xyz="0 0 1"/>
-      <dynamics damping="0.2"/>
+      <!-- <dynamics damping="0.2"/> -->
     </joint>
     <!-- IMU sensor -->
@@ -62,7 +62,7 @@
         <origin xyz="0 0 0" rpy="0 0 0"/>
         <geometry>
-          <box size="0.0000001 0.0000001 0.0000001"/>
-        </geometry>
-        <material name="invisible"/>
+          <box size="0.01 0.01 0.01"/>
+        </geometry>
+        <material name="red"/>
       </visual>
       <inertial>
@@ -78,5 +78,5 @@
       <parent link="chassis_link"/>
       <child link="imu_link"/>
-      <origin xyz="0 0 0" rpy="0 0 0"/>
+      <origin xyz="0 0 0.02" rpy="0 0 0"/>
     </joint>
     <!-- Ultrasonic sensor -->
@@ -180,8 +180,19 @@
     <link name="front_right_wheel">
       <collision>
-        <origin xyz="0 0 0" rpy="${PI/2} 0 ${PI/2}"/>
-        <geometry>
-          <cylinder length="${wheel_len}" radius="${wheel_radius}"/>
-        </geometry>
+        <!-- <geometry>
+          <sphere radius="${wheel_radius}"/>
+        </geometry> -->
+        <origin xyz="0 0 0" rpy="${PI/2} 0 ${PI/2}"/>
+        <geometry>
+          <cylinder length="${wheel_len}" radius="${wheel_radius}"/>
+        </geometry>
+        <surface>
+          <friction>
+            <ode>
+              <mu>1.0</mu>
+              <mu2>0.1</mu2>
+            </ode>
+          </friction>
+        </surface>
       </collision>
       <visual>
@@ -214,8 +225,19 @@
     <link name="front_left_wheel">
       <collision>
-        <origin xyz="0 0 0" rpy="${PI/2} 0 ${PI/2}"/>
-        <geometry>
-          <cylinder length="${wheel_len}" radius="${wheel_radius}"/>
-        </geometry>
+        <!-- <geometry>
+            <sphere radius="${wheel_radius}"/>
+        </geometry> -->
+        <origin xyz="0 0 0" rpy="${PI/2} 0 ${PI/2}"/>
+        <geometry>
+          <cylinder length="${wheel_len}" radius="${wheel_radius}"/>
+        </geometry>
+        <surface>
+          <friction>
+            <ode>
+              <mu>1.0</mu>
+              <mu2>0.1</mu2>
+            </ode>
+          </friction>
+        </surface>
       </collision>
       <visual>
@@ -281,8 +303,19 @@
     <link name="rear_right_wheel">
       <collision>
-        <origin xyz="0 0 0" rpy="${PI/2} 0 ${PI/2}"/>
-        <geometry>
-          <cylinder length="${wheel_len}" radius="${wheel_radius}"/>
-        </geometry>
+        <!-- <geometry>
+            <sphere radius="${wheel_radius}"/>
+        </geometry> -->
+        <origin xyz="0 0 0" rpy="${PI/2} 0 ${PI/2}"/>
+        <geometry>
+          <cylinder length="${wheel_len}" radius="${wheel_radius}"/>
+        </geometry>
+        <surface>
+          <friction>
+            <ode>
+              <mu>1.0</mu>
+              <mu2>0.1</mu2>
+            </ode>
+          </friction>
+        </surface>
       </collision>
       <visual>
@@ -313,25 +346,36 @@
     <!-- rear left wheel -->
     <link name="rear_left_wheel">
-        <collision>
-          <origin xyz="0 0 0" rpy="${PI/2} 0 ${PI/2}"/>
-          <geometry>
-            <cylinder length="${wheel_len}" radius="${wheel_radius}"/>
-          </geometry>
-        </collision>
-        <visual>
-          <origin xyz="0 0 0" rpy="${PI/2} 0 ${PI/2}"/>
-          <geometry>
-            <cylinder length="${wheel_len}" radius="${wheel_radius}"/>
-          </geometry>
-          <material name="black"/>
-        </visual>
-        <inertial>
-          <origin xyz="0 0 0" rpy="${PI/2} 0 ${PI/2}"/>
-          <mass value="${wheel_mass}"/>
-          <inertia
-            ixx="0.0000075875" ixy="0.0" ixz="0.0"
-            iyy="0.0000075875" iyz="0.0"
-            izz="0.000012675"/>
-        </inertial>
+      <collision>
+        <!-- <geometry>
+            <sphere radius="${wheel_radius}"/>
+        </geometry> -->
+        <origin xyz="0 0 0" rpy="${PI/2} 0 ${PI/2}"/>
+        <geometry>
+          <cylinder length="${wheel_len}" radius="${wheel_radius}"/>
+        </geometry>
+        <surface>
+          <friction>
+            <ode>
+              <mu>1.0</mu>
+              <mu2>0.1</mu2>
+            </ode>
+          </friction>
+        </surface>
+      </collision>
+      <visual>
+        <origin xyz="0 0 0" rpy="${PI/2} 0 ${PI/2}"/>
+        <geometry>
+          <cylinder length="${wheel_len}" radius="${wheel_radius}"/>
+        </geometry>
+        <material name="black"/>
+      </visual>
+      <inertial>
+        <origin xyz="0 0 0" rpy="${PI/2} 0 ${PI/2}"/>
+        <mass value="${wheel_mass}"/>
+        <inertia
+          ixx="0.0000075875" ixy="0.0" ixz="0.0"
+          iyy="0.0000075875" iyz="0.0"
+          izz="0.000012675"/>
+      </inertial>
     </link>
     <joint name="rear_left_wheel_joint" type="continuous">

Commit message: fix car not turning in gazebo

File: carlikebot_description/urdf/carlikebot/carlikebot.description.urdf.xacro (robot description, xacro)
@@ -179,4 +179,10 @@
     <!-- front right wheel -->
     <link name="front_right_wheel">
+      <!-- <contact>
+        <lateral_friction value="1.0"/>
+        <rolling_friction value="0.0"/>
+        <stiffness value="30000"/>
+        <damping value="1000"/>
+      </contact> -->
       <collision>
         <!-- <geometry>
@@ -224,4 +230,10 @@
     <!-- front left wheel -->
     <link name="front_left_wheel">
+      <!-- <contact>
+        <lateral_friction value="1.0"/>
+        <rolling_friction value="0.0"/>
+        <stiffness value="30000"/>
+        <damping value="1000"/>
+      </contact> -->
       <collision>
         <!-- <geometry>
@@ -302,4 +314,10 @@
     <!-- rear right wheel -->
     <link name="rear_right_wheel">
+      <!-- <contact>
+        <lateral_friction value="1.0"/>
+        <rolling_friction value="0.0"/>
+        <stiffness value="30000"/>
+        <damping value="1000"/>
+      </contact> -->
       <collision>
         <!-- <geometry>
@@ -346,4 +364,10 @@
     <!-- rear left wheel -->
     <link name="rear_left_wheel">
+      <!-- <contact>
+        <lateral_friction value="1.0"/>
+        <rolling_friction value="0.0"/>
+        <stiffness value="30000"/>
+        <damping value="1000"/>
+      </contact> -->
       <collision>
         <!-- <geometry>

File: carlikebot_description/urdf/carlikebot/carlikebot.gazebo.xacro (robot description, xacro)
@@ -17,4 +17,40 @@
         </xacro:unless>           -->
       </plugin>
+    </gazebo>
+    <gazebo reference="rear_left_wheel">
+      <mu1 value="1.0"/>
+      <mu2 value="0.1"/>
+      <kp value="10000000.0"/>
+      <kd value="1.0"/>
+      <fdir1 value="1 0 0"/>
+      <material>Gazebo/Grey</material>
+      <turnGravityOff>false</turnGravityOff>
+    </gazebo>
+    <gazebo reference="rear_right_wheel">
+      <mu1 value="1.0"/>
+      <mu2 value="0.1"/>
+      <kp value="10000000.0"/>
+      <kd value="1.0"/>
+      <fdir1 value="1 0 0"/>
+      <material>Gazebo/Grey</material>
+      <turnGravityOff>false</turnGravityOff>
+    </gazebo>
+    <gazebo reference="front_left_wheel">
+      <mu1 value="1.0"/>
+      <mu2 value="0.1"/>
+      <kp value="10000000.0"/>
+      <kd value="1.0"/>
+      <fdir1 value="1 0 0"/>
+      <material>Gazebo/Grey</material>
+      <turnGravityOff>false</turnGravityOff>
+    </gazebo>
+    <gazebo reference="front_right_wheel">
+      <mu1 value="1.0"/>
+      <mu2 value="0.1"/>
+      <kp value="10000000.0"/>
+      <kd value="1.0"/>
+      <fdir1 value="1 0 0"/>
+      <material>Gazebo/Grey</material>
+      <turnGravityOff>false</turnGravityOff>
     </gazebo>
     <gazebo reference="imu_link">

File: carlikebot_description/urdf/carlikebot/carlikebot.ros2_control.xacro (robot description, xacro)
@@ -36,4 +36,24 @@
         </state_interface>
       </joint>
+      <joint name="rear_left_wheel_joint">
+        <param name="mimic">front_left_wheel_joint</param>
+        <param name="multiplier">1</param>
+        <state_interface name="velocity">
+          <!-- <param name="initial_value">0.0</param> -->
+        </state_interface>
+        <state_interface name="position">
+          <!-- <param name="initial_value">0.0</param> -->
+        </state_interface>
+      </joint>
+      <joint name="rear_right_wheel_joint">
+        <param name="mimic">front_right_wheel_joint</param>
+        <param name="multiplier">1</param>
+        <state_interface name="velocity">
+          <!-- <param name="initial_value">0.0</param> -->
+        </state_interface>
+        <state_interface name="position">
+          <!-- <param name="initial_value">0.0</param> -->
+        </state_interface>
+      </joint>
       <sensor name="imu_sensor">
         <state_interface name="orientation.x"/>

Commit message: change wheels friction value

File: carlikebot_description/urdf/carlikebot/carlikebot.description.urdf.xacro (robot description, xacro)
@@ -8,5 +8,4 @@
     <xacro:property name="base_length" value="0.195" />
     <xacro:property name="base_height" value="0.002" />
-    <xacro:property name="wheelbase" value="0.145" />
     <xacro:property name="wheel_mass" value="0.024" /> <!-- arbitrary value for wheel mass, I think in Kg -->
     <xacro:property name="wheel_len" value="0.025" />
@@ -197,5 +196,5 @@
             <ode>
               <mu>1.0</mu>
-              <mu2>0.1</mu2>
+              <mu2>1.0</mu2>
             </ode>
           </friction>
@@ -248,5 +247,5 @@
             <ode>
               <mu>1.0</mu>
-              <mu2>0.1</mu2>
+              <mu2>1.0</mu2>
             </ode>
           </friction>

File: carlikebot_description/urdf/carlikebot/carlikebot.gazebo.xacro (robot description, xacro)
@@ -54,10 +54,10 @@
       <turnGravityOff>false</turnGravityOff>
     </gazebo>
-    <gazebo reference="imu_link">
+    <!-- <gazebo reference="imu_link">
       <sensor name="imu_sensor" type="imu">
         <always_on>true</always_on>
         <update_rate>100</update_rate>
       </sensor>
-    </gazebo>
+    </gazebo> -->
     <!-- <gazebo reference="ultrasonic_link">
       <sensor name="ultrasonic" type="ray">
